Commit message: add inertia info

File: description/urdf/open_abcrover_indoor.urdf (robot description, URDF)
Before this commit: robot open_abcrover, 4 links, 3 joints
Links:
- link base_frame: mass None -> 3.258; geometry collision box size=0.293 0.337 0.241; visual mesh filename=package://open_abcrover/description/meshes/base_frame_indoo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
- link left_wheel: mass None -> 0.216; geometry collision box size=0.045 0.152 0.152; visual mesh filename=package://open_abcrover/description/meshes/wheel_left.stl
- link right_wheel: mass None -> 0.216; geometry collision box size=0.045 0.152 0.152; visual mesh filename=package://open_abcrover/description/meshes/wheel_right.stl

Commit message: update robot models:add free casters

File: description/urdf/open_abcrover_indoor.urdf (robot description, URDF)
Before this commit: robot open_abcrover, 4 links, 3 joints
Links:
- added link left_caster_pivot, mass 0.125; collision mesh filename=package://open_abcrover/description/meshes/caster_pivot.stl; visual mesh filename=package://open_abcrover/description/meshes/caster_pivot.stl
- added link left_caster_wheel, mass 0.082; collision mesh filename=package://open_abcrover/description/meshes/caster_wheel.stl; visual mesh filename=package://open_abcrover/description/meshes/caster_wheel.stl
- added link right_caster_pivot, mass 0.125; collision mesh filename=package://open_abcrover/description/meshes/caster_pivot.stl; visual mesh filename=package://open_abcrover/description/meshes/caster_pivot.stl
- added link right_caster_wheel, mass 0.082; collision mesh filename=package://open_abcrover/description/meshes/caster_wheel.stl; visual mesh filename=package://open_abcrover/description/meshes/caster_wheel.stl
- link base_frame: mass 3.258 -> 2.842; geometry collision mesh filename=package://open_abcrover/description/meshes/base_frame_indoo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; visual mesh filename=package://open_abcrover/description/meshes/base_frame_indoo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
- link left_wheel: geometry collision mesh filename=package://open_abcrover/description/meshes/wheel_left.stl; visual mesh filename=package://open_abcrover/description/meshes/wheel_left.stl
- link right_wheel: geometry collision mesh filename=package://open_abcrover/description/meshes/wheel_right.stl; visual mesh filename=package://open_abcrover/description/meshes/wheel_right.stl
Joints:
- added joint base_to_leftcaster_pivot: type continuous, parent base_frame, child left_caster_pivot, origin xyz=0.07 0.10515 -0.0402, axis 0 0 1
- added joint base_to_rightcaster_pivot: type continuous, parent base_frame, child right_caster_pivot, origin xyz=-0.07 0.10515 -0.0402, axis 0 0 1
- added joint left_caster_pivot_to_wheel: type continuous, parent left_caster_pivot, child left_caster_wheel, origin xyz=0 0.02 -0.0555, axis 1 0 0
- added joint right_caster_pivot_to_wheel: type continuous, parent right_caster_pivot, child right_caster_wheel, origin xyz=0 0.02 -0.0555, axis 1 0 0

File: description/urdf/open_abcrover_outdoor.urdf (robot description, URDF)
Before this commit: robot open_abcrover, 4 links, 3 joints
Links:
- added link left_caster_pivot, mass 0.125; collision mesh filename=package://open_abcrover/description/meshes/caster_pivot.stl; visual mesh filename=package://open_abcrover/description/meshes/caster_pivot.stl
- added link left_caster_wheel, mass 0.082; collision mesh filename=package://open_abcrover/description/meshes/caster_wheel.stl; visual mesh filename=package://open_abcrover/description/meshes/caster_wheel.stl
- added link right_caster_pivot, mass 0.125; collision mesh filename=package://open_abcrover/description/meshes/caster_pivot.stl; visual mesh filename=package://open_abcrover/description/meshes/caster_pivot.stl
- added link right_caster_wheel, mass 0.082; collision mesh filename=package://open_abcrover/description/meshes/caster_wheel.stl; visual mesh filename=package://open_abcrover/description/meshes/caster_wheel.stl
- link base_frame: mass None -> 2.802; geometry collision mesh filename=package://open_abcrover/description/meshes/base_frame_outdo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; visual mesh filename=package://open_abcrover/description/meshes/base_frame_outdo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
- link left_wheel: mass None -> 0.216; geometry collision mesh filename=package://open_abcrover/description/meshes/wheel_left.stl; visual mesh filename=package://open_abcrover/description/meshes/wheel_left.stl
- link right_wheel: mass None -> 0.216; geometry collision mesh filename=package://open_abcrover/description/meshes/wheel_right.stl; visual mesh filename=package://open_abcrover/description/meshes/wheel_right.stl
Joints:
- added joint base_to_leftcaster_pivot: type continuous, parent base_frame, child left_caster_pivot, origin xyz=0.07 0.10515 -0.0402, axis 0 0 1
- added joint base_to_rightcaster_pivot: type continuous, parent base_frame, child right_caster_pivot, origin xyz=-0.07 0.10515 -0.0402, axis 0 0 1
- added joint left_caster_pivot_to_wheel: type continuous, parent left_caster_pivot, child left_caster_wheel, origin xyz=0 0.02 -0.0555, axis 1 0 0
- added joint right_caster_pivot_to_wheel: type continuous, parent right_caster_pivot, child right_caster_wheel, origin xyz=0 0.02 -0.0555, axis 1 0 0
